Commit message: adjusted xacro file with revolute joints. got controller working. gains tuned

File: catkin_ws/src/scara_robot/scara_description/urdf/scara.xacro (robot description, xacro)
@@ -23,26 +23,57 @@
   <!-- Base Link -->
   <link name="link1">
-    <visual>
+    <collision>
       <origin xyz="0 0 ${height1/2}" rpy="0 0 0"/>
       <geometry>
    <cylinder length="${height1}" radius="0.2"/>
       </geometry>
+    </collision>
+    <visual>
+      <origin xyz="0 0 ${height1/2}" rpy="0 0 0"/>
+      <geometry>
+   <cylinder length="${height1}" radius="0.2"/>
+      </geometry>
       <material name="orange"/>
     </visual>
-  </link>
-  <joint name="joint1" type="fixed">
+    <inertial>
+      <origin xyz="0 0 ${height1/2}" rpy="0 0 0"/>
+      <mass value="${mass}"/>
+      <inertia
+    ixx="${mass / 12.0 * (width*width + height1*height1)}" ixy="0.0" ixz="0.0"
+    iyy="${mass / 12.0 * (height1*height1 + width*width)}" iyz="0.0"
+    izz="${mass / 12.0 * (width*width + width*width)}"/>
+    </inertial>
+  </link>
+  <joint name="joint1" type="revolute">
     <parent link="link1"/>
     <child link="link2"/>
     <origin xyz="0 0 ${height1 - axel_offset}" rpy="0 0 1.570796"/>
+    <axis xyz="0 0 1"/>
+    <limit effort="100" lower="-1.57" upper="1.57" velocity="1"/>
+    <dynamics damping="0.7"/>
   </joint>
   <!-- Middle Link -->
   <link name="link2">
-    <visual>
+    <collision>
       <origin xyz="0 0 ${height2}" rpy="0 0 0"/>
       <geometry>
    <cylinder length="${height1}" radius="0.2"/>
       </geometry>
+    </collision>
+    <visual>
+      <origin xyz="0 0 ${height2}" rpy="0 0 0"/>
+      <geometry>
+   <cylinder length="${height1}" radius="0.2"/>
+      </geometry>
       <material name="red"/>
     </visual>
+    <inertial>
+      <origin xyz="0 0 ${height2}" rpy="0 0 0"/>
+      <mass value="${mass}"/>
+      <inertia
+    ixx="${mass / 12.0 * (width*width + height2*height2)}" ixy="0.0" ixz="0.0"
+    iyy="${mass / 12.0 * (height2*height2 + width*width)}" iyz="0.0"
+    izz="${mass / 12.0 * (width*width + width*width)}"/>
+    </inertial>
   </link>
   <joint name="joint2" type="fixed">
@@ -52,25 +83,56 @@
   </joint>
   <link name="link3">
-    <visual>
+    <collision>
       <origin xyz="0 0 1.25" rpy="0 0 0"/>
       <geometry>
    <box size="${width} ${width} 2.5"/>
       </geometry>
+    </collision>
+    <visual>
+      <origin xyz="0 0 1.25" rpy="0 0 0"/>
+      <geometry>
+   <box size="${width} ${width} 2.5"/>
+      </geometry>
       <material name="orange"/>
     </visual>
-  </link>
-  <joint name="joint3" type="fixed">
+    <inertial>
+      <origin xyz="0 0 1.25" rpy="0 0 0"/>
+      <mass value="${mass}"/>
+      <inertia
+    ixx="${mass / 12.0 * (width*width + height3*height3)}" ixy="0.0" ixz="0.0"
+    iyy="${mass / 12.0 * (height3*height3 + width*width)}" iyz="0.0"
+    izz="${mass / 12.0 * (width*width + width*width)}"/>
+    </inertial>
+  </link>
+  <joint name="joint3" type="revolute">
     <parent link="link3"/>
     <child link="link4"/>
     <origin xyz="0 1.5 2.5" rpy="1.57 0 0"/>
+    <axis xyz="0 0 1"/>
+    <limit effort="100" lower="-1.57" upper="1.57" velocity="1"/>
+    <dynamics damping="0.7"/>
   </joint>
   <link name="link4">
-    <visual>
+    <collision>
       <origin xyz="0 0 1.5" rpy="0 0 0"/>
       <geometry>
    <cylinder length="1" radius="${width}"/>
       </geometry>
+    </collision>
+    <visual>
+      <origin xyz="0 0 1.5" rpy="0 0 0"/>
+      <geometry>
+   <cylinder length="1" radius="${width}"/>
+      </geometry>
       <material name="blue"/>
     </visual>
+    <inertial>
+      <origin xyz="0 0 1.5" rpy="0 0 0"/>
+      <mass value="${mass}"/>
+      <inertia
+    ixx="${mass / 12.0 * (width*width + height3*height3)}" ixy="0.0" ixz="0.0"
+    iyy="${mass / 12.0 * (height3*height3 + width*width)}" iyz="0.0"
+    izz="${mass / 12.0 * (width*width + width*width)}"/>
+    </inertial>
   </link>
   <joint name="joint4" type="fixed">

Commit message: added PD controller results and steps to run. updated MATLAB plotter

File: catkin_ws/src/scara_robot/scara_description/urdf/scara.xacro (robot description, xacro)
@@ -49,6 +49,6 @@
     <child link="link2"/>
     <origin xyz="0 0 ${height1 - axel_offset}" rpy="0 0 1.570796"/>
-    <axis xyz="0 0 1"/>
-    <limit effort="100" lower="-1.57" upper="1.57" velocity="1"/>
+    <axis xyz="0 0 -1"/>
+    <limit effort="100" lower="-3.14" upper="3.14" velocity="1"/>
     <dynamics damping="0.7"/>
   </joint>
@@ -110,5 +110,5 @@
     <origin xyz="0 1.5 2.5" rpy="1.57 0 0"/>
     <axis xyz="0 0 1"/>
-    <limit effort="100" lower="-1.57" upper="1.57" velocity="1"/>
+    <limit effort="100" lower="-3" upper="3" velocity="1"/>
     <dynamics damping="0.7"/>
   </joint>
